File: connectors.kicad_sch (KiCad schematic)
At the start: 5 parts, among them J1 Conn_01x07_Female, SW1 SW_Push, U10 Payload

Commit message: last commit
Changed lines of the file:
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@@
 (kicad_sch (version 20211123) (generator eeschema)
   (paper "A4")
-  (junction (at 86.995 73.66) (diameter 0) (color 0 0 0 0)
+  (junction (at 185.42 55.88) (diameter 0) (color 0 0 0 0)
+  )
+  (junction (at 195.58 49.53) (diameter 0) (color 0 0 0 0)
   )
   (junction (at 191.135 53.34) (diameter 0) (color 0 0 0 0)
-  )
-  (junction (at 195.58 48.895) (diameter 0) (color 0 0 0 0)
-  )
-  (junction (at 185.42 55.88) (diameter 0) (color 0 0 0 0)
-  )
-  (junction (at 79.375 76.2) (diameter 0) (color 0 0 0 0)
   )
   (junction (at 92.075 84.455) (diameter 0) (color 0 0 0 0)
@@
     (stroke (width 0) (type default) (color 0 0 0 0))
   )
+  (wire (pts (xy 79.375 71.755) (xy 79.375 79.375))
+    (stroke (width 0) (type default) (color 0 0 0 0))
+  )
   (polyline (pts (xy 179.705 42.545) (xy 179.705 69.215))
     (stroke (width 0) (type default) (color 0 0 0 0))
@@
     (stroke (width 0) (type default) (color 0 0 0 0))
   )
+  (wire (pts (xy 195.58 48.895) (xy 195.58 49.53))
+    (stroke (width 0) (type default) (color 0 0 0 0))
+  )
+  (wire (pts (xy 185.42 53.975) (xy 185.42 55.88))
+    (stroke (width 0) (type default) (color 0 0 0 0))
+  )
   (wire (pts (xy 86.36 84.455) (xy 86.36 85.09))
     (stroke (width 0) (type default) (color 0 0 0 0))
   )
-  (wire (pts (xy 79.375 76.2) (xy 79.375 79.375))
+  (wire (pts (xy 191.135 53.34) (xy 191.135 54.61))
     (stroke (width 0) (type default) (color 0 0 0 0))
   )
@@
     (stroke (width 0) (type default) (color 0 0 0 0))
   )
-  (wire (pts (xy 86.995 73.66) (xy 86.995 72.39))
+  (wire (pts (xy 86.995 72.39) (xy 86.995 76.835))
     (stroke (width 0) (type default) (color 0 0 0 0))
   )
@@
     (stroke (width 0) (type default) (color 0 0 0 0))
   )
-  (wire (pts (xy 185.42 53.975) (xy 185.42 55.88))
-    (stroke (width 0) (type default) (color 0 0 0 0))
-  )
   (polyline (pts (xy 179.705 42.545) (xy 229.87 42.545))
     (stroke (width 0) (type default) (color 0 0 0 0))
@@
     (stroke (width 0) (type default) (color 0 0 0 0))
   )
-  (wire (pts (xy 79.375 71.755) (xy 79.375 76.2))
-    (stroke (width 0) (type default) (color 0 0 0 0))
-  )
   (wire (pts (xy 185.42 57.15) (xy 204.47 57.15))
     (stroke (width 0) (type default) (color 0 0 0 0))
   )
-  (wire (pts (xy 191.135 53.34) (xy 191.135 54.61))
-    (stroke (width 0) (type default) (color 0 0 0 0))
-  )
   (polyline (pts (xy 24.765 31.75) (xy 143.51 31.75))
     (stroke (width 0) (type default) (color 0 0 0 0))
@@
     (stroke (width 0) (type default) (color 0 0 0 0))
   )
-  (wire (pts (xy 195.58 48.895) (xy 195.58 52.07))
-    (stroke (width 0) (type default) (color 0 0 0 0))
-  )
-  (wire (pts (xy 86.995 73.66) (xy 86.995 76.835))
+  (wire (pts (xy 195.58 49.53) (xy 195.58 52.07))
     (stroke (width 0) (type default) (color 0 0 0 0))
   )
@@
     (pin "1")
     (pin "2")
+  )
+  (symbol (lib_id "power:PWR_FLAG") (at 185.42 55.88 270) (unit 1)
+    (in_bom yes) (on_board yes) (fields_autoplaced)
+    (property "Reference" "#FLG0103" (id 0) (at 187.325 55.88 0)
+      (effects (font (size 1.27 1.27)) hide)
+    )
+    (property "Value" "PWR_FLAG" (id 1) (at 188.595 55.8799 90)
+      (effects (font (size 1.27 1.27)) (justify left))
+    )
+    (property "Footprint" "" (id 2) (at 185.42 55.88 0)
+      (effects (font (size 1.27 1.27)) hide)
+    )
+    (property "Datasheet" "~" (id 3) (at 185.42 55.88 0)
+      (effects (font (size 1.27 1.27)) hide)
+    )
+    (pin "1")
   )
   (symbol (lib_id "power:+5V") (at 191.135 52.07 0) (unit 1)
@@
     (pin "99")
   )
-  (symbol (lib_id "power:PWR_FLAG") (at 185.42 55.88 270) (unit 1)
-    (in_bom yes) (on_board yes)
-    (property "Reference" "#FLG0103" (id 0) (at 187.325 55.88 0)
-      (effects (font (size 1.27 1.27)) hide)
-    )
-    (property "Value" "PWR_FLAG" (id 1) (at 188.6712 55.88 90)
+  (symbol (lib_id "power:PWR_FLAG") (at 195.58 49.53 270) (unit 1)
+    (in_bom yes) (on_board yes) (fields_autoplaced)
+    (property "Reference" "#FLG0102" (id 0) (at 197.485 49.53 0)
+      (effects (font (size 1.27 1.27)) hide)
+    )
+    (property "Value" "PWR_FLAG" (id 1) (at 198.755 49.5299 90)
       (effects (font (size 1.27 1.27)) (justify left))
     )
-    (property "Footprint" "" (id 2) (at 185.42 55.88 0)
-      (effects (font (size 1.27 1.27)) hide)
-    )
-    (property "Datasheet" "~" (id 3) (at 185.42 55.88 0)
-      (effects (font (size 1.27 1.27)) hide)
-    )
-    (pin "1")
-  )
-  (symbol (lib_id "power:PWR_FLAG") (at 195.58 48.895 270) (unit 1)
-    (in_bom yes) (on_board yes)
-    (property "Reference" "#FLG0101" (id 0) (at 197.485 48.895 0)
-      (effects (font (size 1.27 1.27)) hide)
-    )
-    (property "Value" "PWR_FLAG" (id 1) (at 198.8312 48.895 90)
-      (effects (font (size 1.27 1.27)) (justify left))
-    )
-    (property "Footprint" "" (id 2) (at 195.58 48.895 0)
-      (effects (font (size 1.27 1.27)) hide)
-    )
-    (property "Datasheet" "~" (id 3) (at 195.58 48.895 0)
-      (effects (font (size 1.27 1.27)) hide)
-    )
-    (pin "1")
-  )
-  (symbol (lib_id "power:PWR_FLAG") (at 79.375 76.2 90) (unit 1)
-    (in_bom yes) (on_board yes)
-    (property "Reference" "#FLG0105" (id 0) (at 77.47 76.2 0)
-      (effects (font (size 1.27 1.27)) hide)
-    )
-    (property "Value" "PWR_FLAG" (id 1) (at 83.82 78.105 90)
-      (effects (font (size 1.27 1.27)) (justify left))
-    )
-    (property "Footprint" "" (id 2) (at 79.375 76.2 0)
-      (effects (font (size 1.27 1.27)) hide)
-    )
-    (property "Datasheet" "~" (id 3) (at 79.375 76.2 0)
+    (property "Footprint" "" (id 2) (at 195.58 49.53 0)
+      (effects (font (size 1.27 1.27)) hide)
+    )
+    (property "Datasheet" "~" (id 3) (at 195.58 49.53 0)
       (effects (font (size 1.27 1.27)) hide)
     )
@@
   )
   (symbol (lib_id "power:PWR_FLAG") (at 191.135 53.34 270) (unit 1)
-    (in_bom yes) (on_board yes)
-    (property "Reference" "#FLG0102" (id 0) (at 193.04 53.34 0)
-      (effects (font (size 1.27 1.27)) hide)
-    )
-    (property "Value" "PWR_FLAG" (id 1) (at 194.3862 53.34 90)
+    (in_bom yes) (on_board yes) (fields_autoplaced)
+    (property "Reference" "#FLG0101" (id 0) (at 193.04 53.34 0)
+      (effects (font (size 1.27 1.27)) hide)
+    )
+    (property "Value" "PWR_FLAG" (id 1) (at 194.945 53.3399 90)
       (effects (font (size 1.27 1.27)) (justify left))
     )
@@
       (effects (font (size 1.27 1.27)) hide)
     )
-    (pin "1")
-  )
-  (symbol (lib_id "power:PWR_FLAG") (at 86.995 73.66 90) (unit 1)
-    (in_bom yes) (on_board yes)
-    (property "Reference" "#FLG0104" (id 0) (at 85.09 73.66 0)
-      (effects (font (size 1.27 1.27)) hide)
-    )
-    (property "Value" "PWR_FLAG" (id 1) (at 91.44 75.565 90)
-      (effects (font (size 1.27 1.27)) (justify left))
-    )
-    (property "Footprint" "" (id 2) (at 86.995 73.66 0)
-      (effects (font (size 1.27 1.27)) hide)
-    )
-    (property "Datasheet" "~" (id 3) (at 86.995 73.66 0)
-      (effects (font (size 1.27 1.27)) hide)
-    )
