File: connectors.kicad_sch (KiCad schematic)
At the start: 2 parts, among them J1 Conn_01x07_Female, U2 Payload

Commit message: new uc
Parts:
- added J2: Conn_02x02_Odd_Even, Connector_PinHeader_2.54mm:PinHeader_2x02_P2.54mm_Vertical, symbol Connector_Generic:Conn_02x02_Odd_Even
Connections:
- net +3V3: now also U2.52 (OUT6_3V3-52), J2.3 (Pin_3); no longer U2.51 (51-OUT3_3V3)
- net +5V: now also U2.51 (51-OUT3_5V0), J2.4 (Pin_4); no longer J1.5 (Pin_5), U2.52 (OUT6_5V0-52)
- net SPI-MISO: now reaches U2.10
- net SPI-MOSI: now reaches U2.11 (11-I2C2_SCL)
- net SPI-CS: now reaches U2.12
- net SPI-CLK: now reaches U2.9 (09-I2C2_SDA)
- new net DRV_VM: J2.1 (Pin_1), J2.2 (Pin_2)
- no-connect marks 101 -> 98
